File: coolheat.kicad_sch (KiCad schematic)
At the start: 16 parts, among them J1 SUPPLY, J2 THERMOSTAT 1, J3 THERMOSTAT 2, J4 THERMOSTAT 3, J5 CHAGEOVER, J6 VALVE 1, J7 VALVE 2, J8 VALVE 3, K1 Finder 41.31.8.230.0000, K2 Finder 41.31.8.230.0000, K3 Finder 41.31.8.230.0000, K4 Finder 41.31.8.230.0000

Commit message: hensel case
Parts:
- H1, H2, H3, H4: footprint MountingHole:MountingHole_3.2mm_M3 -> MountingHole:MountingHole_4.3mm_M4
Changed lines of the file:
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@@
 			)
 		)
-		(property "Footprint" "MountingHole:MountingHole_3.2mm_M3"
+		(property "Footprint" "MountingHole:MountingHole_4.3mm_M4"
 			(at 175.26 59.69 0)
 			(effects
@@
 			)
 		)
-		(property "Footprint" "MountingHole:MountingHole_3.2mm_M3"
+		(property "Footprint" "MountingHole:MountingHole_4.3mm_M4"
 			(at 175.26 66.04 0)
 			(effects
@@
 			)
 		)
-		(property "Footprint" "MountingHole:MountingHole_3.2mm_M3"
+		(property "Footprint" "MountingHole:MountingHole_4.3mm_M4"
 			(at 175.26 53.34 0)
 			(effects
@@
 			)
 		)
-		(property "Footprint" "MountingHole:MountingHole_3.2mm_M3"
+		(property "Footprint" "MountingHole:MountingHole_4.3mm_M4"
 			(at 175.26 46.99 0)
 			(effects

Commit message: almost done
Parts:
- X5: renamed from J5; value CHAGEOVER -> CHANGEOVER
- renumbered J1 to X1, J2 to X2, J3 to X3, J4 to X4, J6 to X6, J7 to X7, J8 to X8
Other:
- company: (none) -> SIMON KALLWEIT
- title: (none) -> COOLHEAT CONTROLLER
- moved on the sheet: H1, H2, H3, H4, K1, K2, K3, K4, X1, X2, X3, X4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
